Commit message: upped velocity limits. walking looks more natural now

File: achilles_model_custom/urdf/achilles.urdf (robot description, URDF)
Before this commit: robot achilles, 33 links, 32 joints
Joints:
- joint left_ankle_pitch_joint: limit lower=-1 upper=1 effort=35 velocity=2 -> lower=-1 upper=1 effort=35 velocity=3
- joint left_hip_pitch_joint: limit lower=-1.5 upper=0.5 effort=35.0 velocity=2 -> lower=-1.5 upper=0.5 effort=35.0 velocity=4
- joint left_hip_roll_joint: limit lower=-1 upper=1 effort=70.0 velocity=1 -> lower=-1 upper=1 effort=70.0 velocity=2
- joint left_hip_yaw_joint: limit lower=-1 upper=1 effort=35.0 velocity=2 -> lower=-1 upper=1 effort=35.0 velocity=3
- joint left_knee_pitch_joint: limit lower=0 upper=2 effort=70.0 velocity=1 -> lower=0 upper=2 effort=70.0 velocity=5
- joint right_ankle_pitch_joint: limit lower=-1 upper=1 effort=35 velocity=2 -> lower=-1 upper=1 effort=35 velocity=3
- joint right_hip_pitch_joint: limit lower=-1.5 upper=0.5 effort=35.0 velocity=2 -> lower=-1.5 upper=0.5 effort=35.0 velocity=4
- joint right_hip_roll_joint: limit lower=-1 upper=1 effort=70.0 velocity=1 -> lower=-1 upper=1 effort=70.0 velocity=2
- joint right_hip_yaw_joint: limit lower=-1 upper=1 effort=35.0 velocity=2 -> lower=-1 upper=1 effort=35.0 velocity=3
- joint right_knee_pitch_joint: limit lower=0 upper=2 effort=70.0 velocity=1 -> lower=0 upper=2 effort=70.0 velocity=5
