Commit message: better biped sim walking params. tunned down the PD a lot and that helped

File: g1_model/urdf/g1_hand_full.urdf (robot description, URDF)
Before this commit: robot g1_29dof_with_hand, 57 links, 56 joints
Joints:
- joint left_ankle_pitch_joint: limit lower=-0.87267 upper=0.5236 effort=50 velocity=12 -> lower=-0.87267 upper=0.5236 effort=50 velocity=37
- joint left_ankle_roll_joint: limit lower=-0.2618 upper=0.2618 effort=50 velocity=12 -> lower=-0.2618 upper=0.2618 effort=50 velocity=37
- joint left_elbow_joint: limit lower=-1.0472 upper=2.0944 effort=25 velocity=12 -> lower=-1.0472 upper=2.0944 effort=25 velocity=37
- joint left_hip_pitch_joint: limit lower=-2.5307 upper=2.8798 effort=88 velocity=12 -> lower=-2.5307 upper=2.8798 effort=88 velocity=32
- joint left_hip_roll_joint: limit lower=-0.5236 upper=2.9671 effort=88 velocity=12 -> lower=-0.5236 upper=2.9671 effort=88 velocity=32
- joint left_hip_yaw_joint: limit lower=-2.7576 upper=2.7576 effort=88 velocity=12 -> lower=-2.7576 upper=2.7576 effort=88 velocity=32
- joint left_knee_joint: limit lower=-0.087267 upper=2.8798 effort=139 velocity=12 -> lower=-0.087267 upper=2.8798 effort=139 velocity=20
- joint left_shoulder_pitch_joint: limit lower=-3.0892 upper=2.6704 effort=25 velocity=12 -> lower=-3.0892 upper=2.6704 effort=25 velocity=37
- joint left_shoulder_roll_joint: limit lower=-1.5882 upper=2.2515 effort=25 velocity=12 -> lower=-1.5882 upper=2.2515 effort=25 velocity=37
- joint left_shoulder_yaw_joint: limit lower=-2.618 upper=2.618 effort=25 velocity=12 -> lower=-2.618 upper=2.618 effort=25 velocity=37
- joint left_wrist_roll_joint: limit lower=-1.972222054 upper=1.972222054 effort=25 velocity=12 -> lower=-1.972222054 upper=1.972222054 effort=25 velocity=37
- joint right_ankle_pitch_joint: limit lower=-0.87267 upper=0.5236 effort=50 velocity=12 -> lower=-0.87267 upper=0.5236 effort=50 velocity=37
- joint right_ankle_roll_joint: limit lower=-0.2618 upper=0.2618 effort=50 velocity=12 -> lower=-0.2618 upper=0.2618 effort=50 velocity=37
- joint right_elbow_joint: limit lower=-1.0472 upper=2.0944 effort=25 velocity=12 -> lower=-1.0472 upper=2.0944 effort=25 velocity=37
- joint right_hip_pitch_joint: limit lower=-2.5307 upper=2.8798 effort=88 velocity=12 -> lower=-2.5307 upper=2.8798 effort=88 velocity=32
- joint right_hip_roll_joint: limit lower=-2.9671 upper=0.5236 effort=88 velocity=12 -> lower=-2.9671 upper=0.5236 effort=88 velocity=32
- joint right_hip_yaw_joint: limit lower=-2.7576 upper=2.7576 effort=88 velocity=12 -> lower=-2.7576 upper=2.7576 effort=88 velocity=32
- joint right_knee_joint: limit lower=-0.087267 upper=2.8798 effort=139 velocity=12 -> lower=-0.087267 upper=2.8798 effort=139 velocity=20
- joint right_shoulder_pitch_joint: limit lower=-3.0892 upper=2.6704 effort=25 velocity=12 -> lower=-3.0892 upper=2.6704 effort=25 velocity=37
- joint right_shoulder_roll_joint: limit lower=-2.2515 upper=1.5882 effort=25 velocity=12 -> lower=-2.2515 upper=1.5882 effort=25 velocity=37
- joint right_shoulder_yaw_joint: limit lower=-2.618 upper=2.618 effort=25 velocity=12 -> lower=-2.618 upper=2.618 effort=25 velocity=37
- joint right_wrist_roll_joint: limit lower=-1.972222054 upper=1.972222054 effort=25 velocity=12 -> lower=-1.972222054 upper=1.972222054 effort=25 velocity=37
- joint waist_pitch_joint: limit lower=-0.52 upper=0.52 effort=50 velocity=12 -> lower=-0.52 upper=0.52 effort=50 velocity=37
- joint waist_roll_joint: limit lower=-0.52 upper=0.52 effort=50 velocity=12 -> lower=-0.52 upper=0.52 effort=50 velocity=37
- joint waist_yaw_joint: limit lower=-2.618 upper=2.618 effort=88 velocity=12 -> lower=-2.618 upper=2.618 effort=88 velocity=32
