Commit message: updated the viz urdf to have more accurate hand joint defaults

File: g1_model/urdf/g1_viz.urdf (robot description, URDF)
Before this commit: robot g1_29dof_with_hand, 69 links, 68 joints
Joints:
- joint left_hand_index_0_joint: origin xyz=0.0777 0.0016 0.0285 rpy=0 0 0 -> xyz=0.0777 0.0016 0.0285 rpy=0 0 -1.57
- joint left_hand_index_1_joint: origin xyz=0.0458 0 0 rpy=0 0 0 -> xyz=0.0458 0 0 rpy=0 0 -1.57
- joint left_hand_middle_0_joint: origin xyz=0.0777 0.0016 -0.0285 rpy=0 0 0 -> xyz=0.0777 0.0016 -0.0285 rpy=0 0 -1.57
- joint left_hand_middle_1_joint: origin xyz=0.0458 0 0 rpy=0 0 0 -> xyz=0.0458 0 0 rpy=0 0 -1.57
- joint left_hand_thumb_2_joint: origin xyz=0 -0.0458 0 rpy=0 0 0 -> xyz=0 -0.0458 0 rpy=0 0 1.57
- joint right_hand_index_0_joint: origin xyz=0.0777 -0.0016 0.0285 rpy=0 0 0 -> xyz=0.0777 -0.0016 0.0285 rpy=0 0 1.57
- joint right_hand_index_1_joint: origin xyz=0.0458 0 0 rpy=0 0 0 -> xyz=0.0458 0 0 rpy=0 0 1.57
- joint right_hand_middle_0_joint: origin xyz=0.0777 -0.0016 -0.0285 rpy=0 0 0 -> xyz=0.0777 -0.0016 -0.0285 rpy=0 0 1.57
- joint right_hand_middle_1_joint: origin xyz=0.0458 0 0 rpy=0 0 0 -> xyz=0.0458 0 0 rpy=0 0 1.57
- joint right_hand_thumb_2_joint: origin xyz=0 0.0458 0 rpy=0 0 0 -> xyz=0 0.0458 0 rpy=0 0 -1.57
