Commit message: added config files for the g1

File: g1_model/urdf/g1_hand.urdf (robot description, URDF)
Before this commit: robot g1_29dof_with_hand, 53 links, 52 joints
Links:
- added link left_heel
- added link left_toe
- added link right_heel
- added link right_toe
Joints:
- added joint left_heel_joint: type fixed, parent left_ankle_roll_link, child left_heel, origin xyz=-0.05 0 -0.03 rpy=0 0 0
- added joint left_toe_joint: type fixed, parent left_ankle_roll_link, child left_toe, origin xyz=0.12 0 -0.03 rpy=0 0 0
- added joint right_heel_joint: type fixed, parent right_ankle_roll_link, child right_heel, origin xyz=-0.05 0 -0.03 rpy=0 0 0
- added joint right_toe_joint: type fixed, parent right_ankle_roll_link, child right_toe, origin xyz=0.12 0 -0.03 rpy=0 0 0

Commit message: g1 config files load in without error. urdf updated to be displayed in the viz tool

File: g1_model/urdf/g1_hand.urdf (robot description, URDF)
Before this commit: robot g1_29dof_with_hand, 57 links, 56 joints
Links:
- link head_link: geometry collision mesh filename=package://g1_model/meshes/head_link.STL; visual mesh filename=package://g1_model/meshes/head_link.STL
- link left_ankle_pitch_link: geometry collision mesh filename=package://g1_model/meshes/left_ankle_pitch_link.STL; visual mesh filename=package://g1_model/meshes/left_ankle_pitch_link.STL
- link left_ankle_roll_link: geometry collision sphere radius=0.005; collision sphere radius=0.005
- link left_elbow_link: geometry collision mesh filename=package://g1_model/meshes/left_elbow_link.STL; visual mesh filename=package://g1_model/meshes/left_elbow_link.STL
- link left_hand_index_0_link: geometry collision mesh filename=package://g1_model/meshes/left_hand_index_0_link.STL; visual mesh filename=package://g1_model/meshes/left_hand_index_0_link.STL
- link left_hand_index_1_link: geometry collision mesh filename=package://g1_model/meshes/left_hand_index_1_link.STL; visual mesh filename=package://g1_model/meshes/left_hand_index_1_link.STL
- link left_hand_middle_0_link: geometry collision mesh filename=package://g1_model/meshes/left_hand_middle_0_link.STL; visual mesh filename=package://g1_model/meshes/left_hand_middle_0_link.STL
- link left_hand_middle_1_link: geometry collision mesh filename=package://g1_model/meshes/left_hand_middle_1_link.STL; visual mesh filename=package://g1_model/meshes/left_hand_middle_1_link.STL
- link left_hand_palm_link: geometry collision mesh filename=package://g1_model/meshes/left_hand_palm_link.STL; visual mesh filename=package://g1_model/meshes/left_hand_palm_link.STL
- link left_hand_thumb_0_link: geometry collision mesh filename=package://g1_model/meshes/left_hand_thumb_0_link.STL; visual mesh filename=package://g1_model/meshes/left_hand_thumb_0_link.STL
- link left_hand_thumb_1_link: geometry collision box size=0.02 0.03 0.02; visual mesh filename=package://g1_model/meshes/left_hand_thumb_1_link.STL
- link left_hand_thumb_2_link: geometry collision mesh filename=package://g1_model/meshes/left_hand_thumb_2_link.STL; visual mesh filename=package://g1_model/meshes/left_hand_thumb_2_link.STL
- link left_hip_pitch_link: geometry collision mesh filename=package://g1_model/meshes/left_hip_pitch_link.STL; visual mesh filename=package://g1_model/meshes/left_hip_pitch_link.STL
- link left_hip_roll_link: geometry collision mesh filename=package://g1_model/meshes/left_hip_roll_link.STL; visual mesh filename=package://g1_model/meshes/left_hip_roll_link.STL
- link left_hip_yaw_link: geometry collision mesh filename=package://g1_model/meshes/left_hip_yaw_link.STL; visual mesh filename=package://g1_model/meshes/left_hip_yaw_link.STL
- link left_knee_link: geometry collision mesh filename=package://g1_model/meshes/left_knee_link.STL; visual mesh filename=package://g1_model/meshes/left_knee_link.STL
- link left_shoulder_pitch_link: geometry collision cylinder length=0.05 radius=0.03; visual mesh filename=package://g1_model/meshes/left_shoulder_pitch_link.STL
- link left_shoulder_roll_link: geometry collision cylinder length=0.03 radius=0.03; visual mesh filename=package://g1_model/meshes/left_shoulder_roll_link.STL
- link left_shoulder_yaw_link: geometry collision mesh filename=package://g1_model/meshes/left_shoulder_yaw_link.STL; visual mesh filename=package://g1_model/meshes/left_shoulder_yaw_link.STL
- link left_wrist_pitch_link: geometry collision mesh filename=package://g1_model/meshes/left_wrist_pitch_link.STL; visual mesh filename=package://g1_model/meshes/left_wrist_pitch_link.STL
- link left_wrist_roll_link: geometry collision mesh filename=package://g1_model/meshes/left_wrist_roll_link.STL; visual mesh filename=package://g1_model/meshes/left_wrist_roll_link.STL
- link left_wrist_yaw_link: geometry collision mesh filename=package://g1_model/meshes/left_wrist_yaw_link.STL; visual mesh filename=package://g1_model/meshes/left_wrist_yaw_link.STL
- link logo_link: geometry collision mesh filename=package://g1_model/meshes/logo_link.STL; visual mesh filename=package://g1_model/meshes/logo_link.STL
- link pelvis: geometry visual mesh filename=package://g1_model/meshes/pelvis.STL
- link pelvis_contour_link: geometry collision mesh filename=package://g1_model/meshes/pelvis_contour_link.STL; visual mesh filename=package://g1_model/meshes/pelvis_contour_link.STL
- link right_ankle_pitch_link: geometry collision mesh filename=package://g1_model/meshes/right_ankle_pitch_link.STL; visual mesh filename=package://g1_model/meshes/right_ankle_pitch_link.STL
- link right_ankle_roll_link: geometry collision sphere radius=0.005; collision sphere radius=0.005
- link right_elbow_link: geometry collision mesh filename=package://g1_model/meshes/right_elbow_link.STL; visual mesh filename=package://g1_model/meshes/right_elbow_link.STL
- link right_hand_index_0_link: geometry collision mesh filename=package://g1_model/meshes/right_hand_index_0_link.STL; visual mesh filename=package://g1_model/meshes/right_hand_index_0_link.STL
- link right_hand_index_1_link: geometry collision mesh filename=package://g1_model/meshes/right_hand_index_1_link.STL; visual mesh filename=package://g1_model/meshes/right_hand_index_1_link.STL
- link right_hand_middle_0_link: geometry collision mesh filename=package://g1_model/meshes/right_hand_middle_0_link.STL; visual mesh filename=package://g1_model/meshes/right_hand_middle_0_link.STL
- link right_hand_middle_1_link: geometry collision mesh filename=package://g1_model/meshes/right_hand_middle_1_link.STL; visual mesh filename=package://g1_model/meshes/right_hand_middle_1_link.STL
- link right_hand_palm_link: geometry collision mesh filename=package://g1_model/meshes/right_hand_palm_link.STL; visual mesh filename=package://g1_model/meshes/right_hand_palm_link.STL
- link right_hand_thumb_0_link: geometry collision mesh filename=package://g1_model/meshes/right_hand_thumb_0_link.STL; visual mesh filename=package://g1_model/meshes/right_hand_thumb_0_link.STL
- link right_hand_thumb_1_link: geometry collision box size=0.02 0.03 0.02; visual mesh filename=package://g1_model/meshes/right_hand_thumb_1_link.STL
- link right_hand_thumb_2_link: geometry collision mesh filename=package://g1_model/meshes/right_hand_thumb_2_link.STL; visual mesh filename=package://g1_model/meshes/right_hand_thumb_2_link.STL
- link right_hip_pitch_link: geometry collision mesh filename=package://g1_model/meshes/right_hip_pitch_link.STL; visual mesh filename=package://g1_model/meshes/right_hip_pitch_link.STL
- link right_hip_roll_link: geometry collision mesh filename=package://g1_model/meshes/right_hip_roll_link.STL; visual mesh filename=package://g1_model/meshes/right_hip_roll_link.STL
- link right_hip_yaw_link: geometry collision mesh filename=package://g1_model/meshes/right_hip_yaw_link.STL; visual mesh filename=package://g1_model/meshes/right_hip_yaw_link.STL
- link right_knee_link: geometry collision mesh filename=package://g1_model/meshes/right_knee_link.STL; visual mesh filename=package://g1_model/meshes/right_knee_link.STL
- link right_shoulder_pitch_link: geometry collision cylinder length=0.05 radius=0.03; visual mesh filename=package://g1_model/meshes/right_shoulder_pitch_link.STL
- link right_shoulder_roll_link: geometry collision cylinder length=0.03 radius=0.03; visual mesh filename=package://g1_model/meshes/right_shoulder_roll_link.STL
- link right_shoulder_yaw_link: geometry collision mesh filename=package://g1_model/meshes/right_shoulder_yaw_link.STL; visual mesh filename=package://g1_model/meshes/right_shoulder_yaw_link.STL
- link right_wrist_pitch_link: geometry collision mesh filename=package://g1_model/meshes/right_wrist_pitch_link.STL; visual mesh filename=package://g1_model/meshes/right_wrist_pitch_link.STL
- link right_wrist_roll_link: geometry collision mesh filename=package://g1_model/meshes/right_wrist_roll_link.STL; visual mesh filename=package://g1_model/meshes/right_wrist_roll_link.STL
- link right_wrist_yaw_link: geometry collision mesh filename=package://g1_model/meshes/right_wrist_yaw_link.STL; visual mesh filename=package://g1_model/meshes/right_wrist_yaw_link.STL
- link torso_link: geometry collision mesh filename=package://g1_model/meshes/torso_link.STL; visual mesh filename=package://g1_model/meshes/torso_link.STL
- link waist_roll_link: geometry visual mesh filename=package://g1_model/meshes/waist_roll_link.STL
- link waist_support_link: geometry collision mesh filename=package://g1_model/meshes/waist_support_link.STL; visual mesh filename=package://g1_model/meshes/waist_support_link.STL
- link waist_yaw_link: geometry visual mesh filename=package://g1_model/meshes/waist_yaw_link.STL

Commit message: [wip] working on getting the humanoid to walk. added in the WBC

File: g1_model/urdf/g1_hand.urdf (robot description, URDF)
Before this commit: robot g1_29dof_with_hand, 57 links, 56 joints
Links:
- added link ll_heel
- added link ll_toe
- added link lr_heel
- added link lr_toe
- added link rl_heel
- added link rl_toe
- added link rr_heel
- added link rr_toe
Joints:
- added joint ll_heel_joint: type fixed, parent left_ankle_roll_link, child ll_heel, origin xyz=-0.05 0.025 -0.03 rpy=0 0 0
- added joint ll_toe_joint: type fixed, parent left_ankle_roll_link, child ll_toe, origin xyz=0.12 0.03 -0.03 rpy=0 0 0
- added joint lr_heel_joint: type fixed, parent left_ankle_roll_link, child lr_heel, origin xyz=-0.05 -0.025 -0.03 rpy=0 0 0
- added joint lr_toe_joint: type fixed, parent left_ankle_roll_link, child lr_toe, origin xyz=0.12 -0.03 -0.03 rpy=0 0 0
- added joint rl_heel_joint: type fixed, parent left_ankle_roll_link, child rl_heel, origin xyz=-0.05 0.025 -0.03 rpy=0 0 0
- added joint rl_toe_joint: type fixed, parent left_ankle_roll_link, child rl_toe, origin xyz=0.12 0.03 -0.03 rpy=0 0 0
- added joint rr_heel_joint: type fixed, parent left_ankle_roll_link, child rr_heel, origin xyz=-0.05 -0.025 -0.03 rpy=0 0 0
- added joint rr_toe_joint: type fixed, parent left_ankle_roll_link, child rr_toe, origin xyz=0.12 -0.03 -0.03 rpy=0 0 0

Commit message: added support for using the mocap in the torso. uses the pelvis IMU for the angular velocity. everything looks like it works in sim

File: g1_model/urdf/g1_hand.urdf (robot description, URDF)
Before this commit: robot g1_29dof_with_hand, 67 links, 66 joints
Links:
- removed link imu_link
- added link imu_in_pelvis
- added link imu_in_torso
- added link torso_mocap
Joints:
- removed joint imu_joint
- added joint imu_in_pelvis_joint: type fixed, parent pelvis, child imu_in_pelvis, origin xyz=0.04525 0 -0.08339 rpy=0 0 0
- added joint imu_in_torso_joint: type fixed, parent torso_link, child imu_in_torso, origin xyz=-0.03959 -0.00224 0.13792 rpy=0 0 0
- added joint torso_mocap_joint: type fixed, parent torso_link, child torso_mocap, origin xyz=0 0 0.1 rpy=0 0 0

Commit message: added support for the tracking camera

File: g1_model/urdf/g1_hand.urdf (robot description, URDF)
Before this commit: robot g1_29dof_with_hand, 69 links, 68 joints
Links:
- added link torso_tracking_camera
Joints:
- added joint torso_tracking_camera_joint: type fixed, parent torso_link, child torso_tracking_camera, origin xyz=0 0 0.1 rpy=0 0 0

Commit message: hardware standing with the WBC and camera

File: g1_model/urdf/g1_hand.urdf (robot description, URDF)
Before this commit: robot g1_29dof_with_hand, 70 links, 69 joints
Joints:
- joint torso_tracking_camera_joint: origin xyz=0 0 0.1 rpy=0 0 0 -> xyz=0.085725 0 0.2413 rpy=0.02 -0.08 0
