Commit message: changes so the viz will display the robot

File: go2_model/urdf/go2_description.urdf (robot description, URDF)
Before this commit: robot go2_description, 41 links, 40 joints
Links:
- removed link base
- added link base_link
- added link torso, mass 6.921; collision box size=0.3762 0.0935 0.114; visual mesh filename=package://go2_description/meshes/trunk.dae
Joints:
- added joint base_to_torso_joint: type fixed, parent base_link, child torso, origin xyz=0 0 0 rpy=0 0 0
- joint FL_hip_joint: parent base -> torso
- joint FL_hip_rotor_joint: parent base -> torso
- joint FR_hip_joint: parent base -> torso
- joint FR_hip_rotor_joint: parent base -> torso
- joint Head_upper_joint: parent base -> torso
- joint RL_hip_joint: parent base -> torso
- joint RL_hip_rotor_joint: parent base -> torso
- joint RR_hip_joint: parent base -> torso
- joint RR_hip_rotor_joint: parent base -> torso
- joint imu_joint: parent base -> torso
- joint radar_joint: parent base -> torso

Commit message: added joystick support. started parsing joystick commands

File: go2_model/urdf/go2_description.urdf (robot description, URDF)
Before this commit: robot go2_description, 42 links, 41 joints
Joints:
- joint FL_calf_joint: limit lower=-2.7227 upper=-0.83776 effort=45.43 velocity=3 -> lower=-2.7227 upper=-0.83776 effort=45.43 velocity=6
- joint FL_hip_joint: limit lower=-1.0472 upper=1.0472 effort=23.7 velocity=5 -> lower=-1.0472 upper=1.0472 effort=23.7 velocity=6
- joint FL_thigh_joint: limit lower=-1.5708 upper=3.4907 effort=23.7 velocity=5 -> lower=-1.5708 upper=3.4907 effort=23.7 velocity=6
- joint FR_calf_joint: limit lower=-2.7227 upper=-0.83776 effort=45.43 velocity=3 -> lower=-2.7227 upper=-0.83776 effort=45.43 velocity=6
- joint FR_hip_joint: limit lower=-1.0472 upper=1.0472 effort=23.7 velocity=5 -> lower=-1.0472 upper=1.0472 effort=23.7 velocity=6
- joint FR_thigh_joint: limit lower=-1.5708 upper=3.4907 effort=23.7 velocity=5 -> lower=-1.5708 upper=3.4907 effort=23.7 velocity=6
- joint RL_calf_joint: limit lower=-2.7227 upper=-0.83776 effort=45.43 velocity=3 -> lower=-2.7227 upper=-0.83776 effort=45.43 velocity=6
- joint RL_hip_joint: limit lower=-1.0472 upper=1.0472 effort=23.7 velocity=5 -> lower=-1.0472 upper=1.0472 effort=23.7 velocity=6
- joint RL_thigh_joint: limit lower=-0.5236 upper=4.5379 effort=23.7 velocity=5 -> lower=-0.5236 upper=4.5379 effort=23.7 velocity=6
- joint RR_calf_joint: limit lower=-2.7227 upper=-0.83776 effort=45.43 velocity=3 -> lower=-2.7227 upper=-0.83776 effort=45.43 velocity=6
- joint RR_hip_joint: limit lower=-1.0472 upper=1.0472 effort=23.7 velocity=5 -> lower=-1.0472 upper=1.0472 effort=23.7 velocity=6
- joint RR_thigh_joint: limit lower=-0.5236 upper=4.5379 effort=23.7 velocity=5 -> lower=-0.5236 upper=4.5379 effort=23.7 velocity=6

Commit message: upped velocity limits on the joints in the go2. was able to not tip with commanding 1m/s, just need to slow down slowly sometimes.

File: go2_model/urdf/go2_description.urdf (robot description, URDF)
Before this commit: robot go2_description, 42 links, 41 joints
Joints:
- joint FL_calf_joint: limit lower=-2.7227 upper=-0.83776 effort=45.43 velocity=6 -> lower=-2.7227 upper=-0.83776 effort=45.43 velocity=10
- joint FL_hip_joint: limit lower=-1.0472 upper=1.0472 effort=23.7 velocity=6 -> lower=-1.0472 upper=1.0472 effort=23.7 velocity=10
- joint FL_thigh_joint: limit lower=-1.5708 upper=3.4907 effort=23.7 velocity=6 -> lower=-1.5708 upper=3.4907 effort=23.7 velocity=10
- joint FR_calf_joint: limit lower=-2.7227 upper=-0.83776 effort=45.43 velocity=6 -> lower=-2.7227 upper=-0.83776 effort=45.43 velocity=10
- joint FR_hip_joint: limit lower=-1.0472 upper=1.0472 effort=23.7 velocity=6 -> lower=-1.0472 upper=1.0472 effort=23.7 velocity=10
- joint FR_thigh_joint: limit lower=-1.5708 upper=3.4907 effort=23.7 velocity=6 -> lower=-1.5708 upper=3.4907 effort=23.7 velocity=10
- joint RL_calf_joint: limit lower=-2.7227 upper=-0.83776 effort=45.43 velocity=6 -> lower=-2.7227 upper=-0.83776 effort=45.43 velocity=10
- joint RL_hip_joint: limit lower=-1.0472 upper=1.0472 effort=23.7 velocity=6 -> lower=-1.0472 upper=1.0472 effort=23.7 velocity=10
- joint RL_thigh_joint: limit lower=-0.5236 upper=4.5379 effort=23.7 velocity=6 -> lower=-0.5236 upper=4.5379 effort=23.7 velocity=10
- joint RR_calf_joint: limit lower=-2.7227 upper=-0.83776 effort=45.43 velocity=6 -> lower=-2.7227 upper=-0.83776 effort=45.43 velocity=10
- joint RR_hip_joint: limit lower=-1.0472 upper=1.0472 effort=23.7 velocity=6 -> lower=-1.0472 upper=1.0472 effort=23.7 velocity=10
- joint RR_thigh_joint: limit lower=-0.5236 upper=4.5379 effort=23.7 velocity=6 -> lower=-0.5236 upper=4.5379 effort=23.7 velocity=10

Commit message: added the camera to the quadruped in sim

File: go2_model/urdf/go2_description.urdf (robot description, URDF)
Before this commit: robot go2_description, 42 links, 41 joints
Links:
- added link torso_tracking_camera
Joints:
- added joint base_tracking_camera_joint: type fixed, parent torso, child torso_tracking_camera, origin xyz=-0.0635 -0.12 -0.01 rpy=0.0 0.0 1.57079

Commit message: [WIP] looks like the camera frames are sorted out on hardware

File: go2_model/urdf/go2_description.urdf (robot description, URDF)
Before this commit: robot go2_description, 43 links, 42 joints
Joints:
- joint base_tracking_camera_joint: origin xyz=-0.0635 -0.12 -0.01 rpy=0.0 0.0 1.57079 -> xyz=-0.0635 -0.12 -0.01 rpy=0.0 3.14159 1.57079

Commit message: good standing on the quad with MPC. could vary the base height

File: go2_model/urdf/go2_description.urdf (robot description, URDF)
Before this commit: robot go2_description, 43 links, 42 joints
Links:
- added link torso_tracking_camera_vel_frame
Joints:
- added joint base_tracking_camera_vel_frame_joint: type fixed, parent torso, child torso_tracking_camera_vel_frame, origin xyz=-0.0635 -0.12 -0.01 rpy=0.0 0 -1.57079

Commit message: gap crossing works on hardware with the terrain

File: go2_model/urdf/go2_description.urdf (robot description, URDF)
Before this commit: robot go2_description, 44 links, 43 joints
Links:
- added link torso_mocap
Joints:
- added joint torso_mocap_joint: type fixed, parent torso, child torso_mocap, origin xyz=0 0 0 rpy=0.0 0 0
